File: shaghayeghs-keyboard.kicad_pcb (KiCad board)
At the start: 2 copper layers, 80 x 119 mm, 51 parts, among them J1 DISPLAY, M2 MountingHole_2.2mm_M2, SW1 SW_Push, SW10 SW_Push, SW11 SW_Push, SW12 SW_Push, SW13 SW_Push, SW14 SW_Push, SW15 RotaryEncoder_Switch, SW16 RotaryEncoder_Switch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

Commit message: fixes bad diod footprints
Parts:
- removed M2 (x4): MountingHole_2.2mm_M2, MountingHole:MountingHole_2.2mm_M2
- D1, D10, D11, D12, D13, D14, D2, D3, D4, D5, D6, D7, D8, D9: footprint Diode_SMD:D_1206_3216Metric -> Diode_SMD:D_SOD-123
Connections:
- U1 pad 22: Net-(U1-RST) -> unconnected-(U1-RST-Pad22)
