File: shaghayeghs-keyboard.kicad_sch (KiCad schematic)
At the start: 46 parts, among them J1 DISPLAY, SW1 SW_Push, SW10 SW_Push, SW11 SW_Push, SW12 SW_Push, SW13 SW_Push, SW14 SW_Push, SW15 RotaryEncoder_Switch, SW16 RotaryEncoder_Switch, SW2 SW_Push, SW3 SW_Push, SW4 SW_Push, SW5 SW_Push, SW6 SW_Push, SW7 SW_Push, SW8 SW_Push, SW9 SW_Push, U1 Sparkfun_Pro_Micro

Commit message: fixes bad diod footprints
Parts:
- D1, D10, D11, D12, D13, D14, D2, D3, D4, D5, D6, D7, D8, D9: footprint Diode_SMD:D_1206_3216Metric -> Diode_SMD:D_SOD-123
Changed lines of the file:
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@@
 			)
 		)
-		(property "Footprint" "Diode_SMD:D_1206_3216Metric"
+		(property "Footprint" "Diode_SMD:D_SOD-123"
 			(at 250.825 109.22 0)
 			(effects
@@
 			)
 		)
-		(property "Footprint" "Diode_SMD:D_1206_3216Metric"
+		(property "Footprint" "Diode_SMD:D_SOD-123"
 			(at 234.315 128.27 0)
 			(effects
@@
 			)
 		)
-		(property "Footprint" "Diode_SMD:D_1206_3216Metric"
+		(property "Footprint" "Diode_SMD:D_SOD-123"
 			(at 234.315 148.59 0)
 			(effects
@@
 			)
 		)
-		(property "Footprint" "Diode_SMD:D_1206_3216Metric"
+		(property "Footprint" "Diode_SMD:D_SOD-123"
 			(at 201.295 149.86 0)
 			(effects
@@
 			)
 		)
-		(property "Footprint" "Diode_SMD:D_1206_3216Metric"
+		(property "Footprint" "Diode_SMD:D_SOD-123"
 			(at 234.315 90.17 0)
 			(effects
@@
 			)
 		)
-		(property "Footprint" "Diode_SMD:D_1206_3216Metric"
+		(property "Footprint" "Diode_SMD:D_SOD-123"
 			(at 201.295 109.22 0)
 			(effects
@@
 			)
 		)
-		(property "Footprint" "Diode_SMD:D_1206_3216Metric"
+		(property "Footprint" "Diode_SMD:D_SOD-123"
 			(at 201.295 90.17 0)
 			(effects
@@
 			)
 		)
-		(property "Footprint" "Diode_SMD:D_1206_3216Metric"
+		(property "Footprint" "Diode_SMD:D_SOD-123"
 			(at 250.825 148.59 0)
 			(effects
@@
 			)
 		)
-		(property "Footprint" "Diode_SMD:D_1206_3216Metric"
+		(property "Footprint" "Diode_SMD:D_SOD-123"
 			(at 217.805 90.17 0)
 			(effects
@@
 			)
 		)
-		(property "Footprint" "Diode_SMD:D_1206_3216Metric"
+		(property "Footprint" "Diode_SMD:D_SOD-123"
 			(at 217.805 109.22 0)
 			(effects
@@
 			)
 		)
-		(property "Footprint" "Diode_SMD:D_1206_3216Metric"
+		(property "Footprint" "Diode_SMD:D_SOD-123"
 			(at 234.315 109.22 0)
 			(effects
@@
 			)
 		)
-		(property "Footprint" "Diode_SMD:D_1206_3216Metric"
+		(property "Footprint" "Diode_SMD:D_SOD-123"
 			(at 217.805 128.27 0)
 			(effects
@@
 			)
 		)
-		(property "Footprint" "Diode_SMD:D_1206_3216Metric"
+		(property "Footprint" "Diode_SMD:D_SOD-123"
 			(at 201.295 128.27 0)
 			(effects
@@
 			)
 		)
-		(property "Footprint" "Diode_SMD:D_1206_3216Metric"
+		(property "Footprint" "Diode_SMD:D_SOD-123"
 			(at 250.825 90.17 0)
 			(effects

Commit message: First STM32 design
Parts:
- removed U1: Sparkfun_Pro_Micro, Arduino:Sparkfun_Pro_Micro, symbol Arduino:Sparkfun_Pro_Micro
- added C1: 10u, Capacitor_SMD:C_1206_3216Metric, symbol Device:C
- added C10, C12: 2.2u, Capacitor_SMD:C_0805_2012Metric, symbol Device:C
- added C11, C13, C14, C15, C16, C5, C7: 100n, Capacitor_SMD:C_0603_1608Metric, symbol Device:C
- added C17, C18: 1u, Capacitor_SMD:C_0603_1608Metric, symbol Device:C
- added C2: 4.7nF, Capacitor_SMD:C_0603_1608Metric, symbol Device:C
- added C3: 22u, Capacitor_SMD:C_1206_3216Metric, symbol Device:C
- added C4, C8: 4.7u, Capacitor_SMD:C_0805_2012Metric, symbol Device:C
- added C6, C9: 18p, Capacitor_SMD:C_0603_1608Metric, symbol Device:C
- added D1: USBLC6-2SC6, digikey-footprints:SOT23-6L, symbol dk_TVS-Diodes:USBLC6-2SC6
- added D2: ON, LED_SMD:LED_Kingbright_APHBM2012_2x1.25mm, symbol Device:LED_Dual_AKKA
- added F1: Fuse, Resistor_SMD:R_1206_3216Metric, symbol Device:Fuse
- added FB1: FerriteBead, Resistor_SMD:R_0603_1608Metric, symbol Device:FerriteBead
- added H1, H2, H3, H4: MountingHole, MountingHole:MountingHole_2.2mm_M2, symbol Mechanical:MountingHole
- added J1: USB_C_Receptacle_USB2.0_16P, Connector_USB:USB_C_Receptacle_GCT_USB4105-xx-A_16P_TopMnt_Horizontal, symbol Connector:USB_C_Receptacle_USB2.0_16P
- added J2: Conn_02x05_Odd_Even, Connector_PinSocket_2.54mm:PinSocket_2x05_P2.54mm_Vertical, symbol Connector_Generic:Conn_02x05_Odd_Even
- added J4: Conn_01x03_Pin, Connector_PinSocket_2.54mm:PinSocket_1x03_P2.54mm_Vertical, symbol Connector:Conn_01x03_Pin
- added J5: UART, Connector_PinSocket_2.54mm:PinSocket_1x03_P2.54mm_Vertical, symbol Connector:Conn_01x03_Pin
- added Q1: SS8050, Package_TO_SOT_SMD:SOT-23, symbol Transistor_BJT:SS8050
- added R10: 10K, Resistor_SMD:R_0603_1608Metric, symbol Device:R
- added R24, R25, R26, R27: 4K7, Resistor_SMD:R_0805_2012Metric, symbol Device:R
- added R5, R9: 0R, Resistor_SMD:R_0603_1608Metric, symbol Device:R
- added R6, R7: 5.1K, Resistor_SMD:R_0603_1608Metric, symbol Device:R
- added R8: 1R2, Resistor_SMD:R_0603_1608Metric, symbol Device:R
- added RN2: 10K, Resistor_SMD:R_Array_Convex_4x0402, symbol Device:R_Pack04
- added SW1: Reset, Button_Switch_SMD:SW_SPST_B3U-1000P, symbol Switch:SW_Push
- added SW19: Reset, Library:Tactile Tact Key right angled - Aliexpress, symbol Switch:SW_Push
- added SW2: Boot, Button_Switch_SMD:SW_SPST_B3U-1000P, symbol Switch:SW_Push
- added U1: AMS1117-3.3, Package_TO_SOT_SMD:SOT-223-3_TabPin2, symbol Regulator_Linear:AMS1117-3.3
- added U2: STM32H523CCTx, Package_QFP:LQFP-48_7x7mm_P0.5mm, symbol MCU_ST_STM32H5:STM32H523CCTx
- added U3: ATtiny804-SS, Package_SO:SOIC-14_3.9x8.7mm_P1.27mm, symbol MCU_Microchip_ATtiny:ATtiny804-SS
- added Y1: 16MHz, Crystal:Crystal_SMD_3225-4Pin_3.2x2.5mm, symbol Device:Crystal_GND24
- R1: value 10K -> 1M; footprint Resistor_SMD:R_1206_3216Metric -> Resistor_SMD:R_0603_1608Metric
- R11: value 5K -> 10K; footprint Resistor_SMD:R_1206_3216Metric -> Resistor_SMD:R_0603_1608Metric
- R12: footprint Resistor_SMD:R_1206_3216Metric -> Resistor_SMD:R_0603_1608Metric
- R13: value 10K -> 47R; footprint Resistor_SMD:R_1206_3216Metric -> Resistor_SMD:R_0603_1608Metric
- R14: renamed from R6; footprint Resistor_SMD:R_1206_3216Metric -> Resistor_SMD:R_0603_1608Metric
- R15: renamed from R7; footprint Resistor_SMD:R_1206_3216Metric -> Resistor_SMD:R_0603_1608Metric
- R16: renamed from R8; footprint Resistor_SMD:R_1206_3216Metric -> Resistor_SMD:R_0603_1608Metric
- R18: renamed from R9; footprint Resistor_SMD:R_1206_3216Metric -> Resistor_SMD:R_0603_1608Metric
- R19: renamed from R10; footprint Resistor_SMD:R_1206_3216Metric -> Resistor_SMD:R_0603_1608Metric
- R2: value 10K -> 1R5; footprint Resistor_SMD:R_1206_3216Metric -> Resistor_SMD:R_0603_1608Metric
- R3: value 10K -> 33K; footprint Resistor_SMD:R_1206_3216Metric -> Resistor_SMD:R_0603_1608Metric
- R4: value 10K -> 75K; footprint Resistor_SMD:R_1206_3216Metric -> Resistor_SMD:R_0603_1608Metric
- renumbered D3 to D10, D7 to D11, D11 to D12, D4 to D14, D8 to D15, D14 to D16, D1 to D3, D5 to D4, D9 to D5, D12 to D6, D2 to D7, D6 to D8, D10 to D9, J1 to J3, R5 to R17, SW16 to SW10, SW3 to SW11, SW7 to SW12, SW11 to SW13, SW13 to SW14, SW4 to SW16, SW8 to SW17, SW14 to SW18, SW1 to SW3, SW5 to SW4, SW9 to SW5, SW12 to SW6, SW2 to SW7, SW6 to SW8, SW10 to SW9
Connections:
- net Col1: now also SW3.2, SW4.2, SW5.2, SW6.2, RN2.1 (R1.1), U2.18 (PB0); no longer R1.1
- net Col2: now also SW7.2, SW8.2, SW9.2, RN2.2 (R2.1), U2.19 (PB1); no longer R2.1
- net Col3: now also SW11.2, SW12.2, SW13.2, SW14.2, RN2.3 (R3.1), U2.20 (PB2); no longer R3.1
- net Col4: now also SW16.2, SW17.2, SW18.2, RN2.4 (R4.1), U2.39 (PB3(JTDO); no longer R4.1
- net GND: now also R1.1, R11.1, R4.2, C1.2, C10.2, C11.1, C12.2, C13.1, C14.1, C15.1, C16.1, C17.1, C18.1, C2.1, C3.2, C4.1, C5.1, C6.2, C7.2, C8.1, C9.2, D1.2, D2.2 (K1), D2.3 (K2), J1.A1 (GND), J1.A12 (GND), J1.B1 (GND), J1.B12 (GND), J2.5 (Pin_5), J2.6 (Pin_6), J4.1 (Pin_1), J5.3 (Pin_3), Q1.2 (E), R6.2, R7.2, SW1.1, SW19.1, U1.1 (GND), U2.23 (VSS), U2.35 (VSS), U2.47 (VSS), U2.8 (VSSA), U3.14 (GND), Y1.2, Y1.4
- net Row1: now also U2.41 (PB5)
- net Row2: now also U2.42 (PB6)
- net Row3: now also U2.43 (PB7)
- net Row4: now also U2.45 (PB8)
- net at SW15.S2: now also U3.4 (PA6); no longer R11.2
- net at SW10.S2: now also U3.13 (PA3); no longer R12.1
- net A1 renamed 5WAY_SW
- net 5WAY_SW: now also U2.10 (PA0)
- removed net A2: R11.1, R12.2, R13.2
- net CLK renamed OLED_I2C_SCL
- net OLED_I2C_SCL: now also R24.1, U2.21 (PB10)
- net E1_A: no longer names the net of SW15.A
- net E1_A: now also U3.2 (PA4)
- net E1_B: no longer names the net of SW15.B
- net E1_B: now also U3.3 (PA5)
- net E2_A: no longer names the net of SW10.A
- net E2_A: now also U3.11 (PA1)
- net E2_B: no longer names the net of SW10.B
- net E2_B: now also U3.12 (PA2)
- net SDA renamed OLED_I2C_SDA
- net OLED_I2C_SDA: now also R25.2, U2.25 (PB12)
- net VCC renamed +3.3V
- net +3.3V: now also R12.1, R13.2, C11.2, C13.2, C14.2, C15.2, C18.2, C3.1, C8.2, J2.7 (Pin_7), J2.8 (Pin_8), J4.3 (Pin_3), Q1.1 (B), R10.1, R24.2, R25.1, R26.1, R27.2, R8.1, RN2.5 (R4.2), RN2.6 (R3.2), RN2.7 (R2.2), RN2.8 (R1.2), U1.2 (VO), U2.1 (VBAT), U2.24 (VDD), U2.36 (VDD), U2.48 (VDD), U3.1 (VCC); no longer R13.1
- new net: J1.A5 (CC1), R6.1
- new net: J1.B5 (CC2), R7.1
- new net: D1.4, R5.1
- new net: D1.5, FB1.1
- new net: D1.6, R9.2
- new net: D2.1 (A1), Q1.3 (C), R2.1
- new net: R10.2, SW2.2
- new net: D2.4 (A2), R8.2
- new net +3.3VA: C16.2, C17.2, R13.1, U2.9 (VDDA)
- new net BOOT: R11.2, SW2.1, U2.44 (BOOT0)
- new net DP+: D1.3, J1.A6 (D+), J1.B6 (D+)
- new net DP-: D1.1, J1.A7 (D-), J1.B7 (D-)
- new net HSE_IN: C6.1, U2.5 (PH0), Y1.1
- new net HSE_OUT: C9.1, U2.6 (PH1), Y1.3
- new net I2C_SCL: R27.1, U2.29 (PA8), U3.9 (PB0)
- new net I2C_SDA: R26.2, U2.40 (PB4(NJTRST)), U3.8 (PB1)
- new net NRST: C7.1, J2.1 (Pin_1), R12.2, SW1.2, SW19.2, U2.7 (NRST)
- new net RX: J5.1 (Pin_1), U2.13 (PA3)
- new net SHILD: C2.2, J1.S1 (SHIELD), R1.2
- new net SWDCLK: J2.2 (Pin_2), U2.37 (PA14(JTCK)
- new net SWDIO: J2.4 (Pin_4), U2.34 (PA13(JTMS)
- new net TX: J5.2 (Pin_2), U2.12 (PA2)
- new net UDPI: J4.2 (Pin_2), U3.10 (~{RESET}/PA0)
- new net USB+: R5.2, U2.33 (PA12)
- new net USB-: R9.1, U2.32 (PA11)
- new net USB_V: F1.2, J1.A4 (VBUS), J1.A9 (VBUS), J1.B4 (VBUS), J1.B9 (VBUS)
- new net VBUS: C1.1, C4.2, C5.2, F1.1, FB1.2, R2.2, R3.2, U1.3 (VI)
- new net VBUS_SENSING: R3.1, R4.1, U2.30 (PA9)
- new net VCAP1: C10.1, U2.22 (VCAP)
- new net VCAP2: C12.1, U2.46 (VCAP)
- no-connect marks 4 -> 21
Other:
- note added: "I2Cs"
- note added: "MCU"
- note added: "Mounting holes"
- note added: "PWR Flags"
- note added: "USB + ESD Protection"
- note added: "Voltage Regulation"
- note removed: "Power lines"
- title: Arduino pro micro based macro keyboard -> Macro keyboard based on STM32H523
- moved on the sheet: D10, D11, D12, D13, D14, D15, D16, D3, D4, D5, D6, D7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
